File: Dattalogger_Board.kicad_pcb (KiCad board)
At the start: 2 copper layers, 0 parts

Commit message: Committing local changes before merge
Parts:
- added BT1: Battery, Connector_PinHeader_2.54mm:PinHeader_2x01_P2.54mm_Vertical, F.Cu at (132.1, 73.7)
- added C1: 0.1uF, Capacitor_SMD:C_0805_2012Metric, F.Cu at (148.0, 66.2)
- added C2: 22pF, Capacitor_SMD:C_0805_2012Metric, F.Cu at (161.3, 83.8)
- added C3: 22pF, Capacitor_SMD:C_0805_2012Metric, F.Cu at (152.4, 66.0)
- added C4: 0.1uF, Capacitor_SMD:C_0805_2012Metric, F.Cu at (161.3, 87.0)
- added C5: 100nF, Capacitor_SMD:C_0805_2012Metric, F.Cu at (156.8, 66.0)
- added D1: LED, LED_SMD:LED_0805_2012Metric, F.Cu at (165.7, 66.0)
- added D2: LED, LED_SMD:LED_0805_2012Metric, F.Cu at (161.9, 66.0)
- added H1: MountingHole, MountingHole:MountingHole_2.1mm, F.Cu at (129.5, 63.5)
- added H2: MountingHole, MountingHole:MountingHole_2.1mm, F.Cu at (129.5, 94.0)
- added H3: MountingHole, MountingHole:MountingHole_2.1mm, F.Cu at (175.3, 63.5)
- added H4: MountingHole, MountingHole:MountingHole_2.1mm, F.Cu at (175.3, 94.0)
- added J1: Conn_01x04_Pin, Connector_PinHeader_2.54mm:PinHeader_1x04_P2.54mm_Vertical, F.Cu at (172.7, 79.4)
- added J2: Conn_01x04_Pin, Connector_PinHeader_2.54mm:PinHeader_1x04_P2.54mm_Vertical, F.Cu at (161.3, 91.4)
- added J3: Conn_02x03_Odd_Even, Connector_PinHeader_2.54mm:PinHeader_2x03_P2.54mm_Vertical, F.Cu at (170.2, 69.2)
- added J4: Conn_01x09_Pin, Connector_PinHeader_2.54mm:PinHeader_1x09_P2.54mm_Vertical, F.Cu at (134.6, 91.4)
- added Majed: LOGO, Library2:MajedDev, B.Cu at (160.7, 76.2)
- added R1: 10K, Resistor_SMD:R_0805_2012Metric, F.Cu at (137.8, 87.0)
- added R2: 10K, Resistor_SMD:R_0805_2012Metric, F.Cu at (141.6, 87.0)
- added R3: 4.7K, Resistor_SMD:R_0805_2012Metric, F.Cu at (161.9, 76.2)
- added R4: 4.7K, Resistor_SMD:R_0805_2012Metric, F.Cu at (161.9, 73.0)
- added R5: 330, Resistor_SMD:R_0805_2012Metric, F.Cu at (161.9, 69.8)
- added R6: 10K, Resistor_SMD:R_0805_2012Metric, F.Cu at (165.7, 73.0)
- added R7: 330, Resistor_SMD:R_0805_2012Metric, F.Cu at (165.7, 69.8)
- added U1: 24LC1025, Package_SO:SOIC-8_5.23x5.23mm_P1.27mm, F.Cu at (140.3, 75.6)
- added U2: DS1337S_, Project_Libraries:SOIC127P600X175-8N, F.Cu at (140.3, 82.5)
- added U3: 24LC1025, Package_SO:SOIC-8_5.23x5.23mm_P1.27mm, F.Cu at (140.3, 67.9)
- added U4: ATMega328P-AU, Project_Libraries:QFP80P900X900X120-32N, F.Cu at (152.4, 76.8)
- added Y1: 32.768 KHz, Crystal:Crystal_SMD_5032-2Pin_5.0x3.2mm_HandSoldering, F.Cu at (132.1, 83.2)
- added Y2: 16 MHz, Crystal:Crystal_SMD_5032-2Pin_5.0x3.2mm_HandSoldering, F.Cu at (152.4, 86.4)
Routing:
- net /Vcc: track 0.00 -> 221.0 mm, vias 0 -> 7
- net GND: track 0.00 -> 185.0 mm, vias 0 -> 5
- net /SCK: track 0.00 -> 99.2 mm, vias 0 -> 3
- net /SDA: track 0.00 -> 64.3 mm, vias 0 -> 4
- net Net-(U4-PB7): track 0.00 -> 31.5 mm, vias 0 -> 2
- net /TX: track 0.00 -> 29.0 mm, vias 0 -> 1
- net /D2: track 0.00 -> 27.4 mm, vias 0 -> 1
- net /RX: track 0.00 -> 27.1 mm, vias 0 -> 1
- net /MOSI: track 0.00 -> 24.8 mm
- net /D3: track 0.00 -> 24.6 mm
- net Net-(U4-PB6): track 0.00 -> 24.2 mm
- net /MISO: track 0.00 -> 23.7 mm, vias 0 -> 1
- net /RESET: track 0.00 -> 22.5 mm, vias 0 -> 2
- net /D4: track 0.00 -> 22.4 mm
- net Net-(U4-AREF): track 0.00 -> 21.1 mm, vias 0 -> 2
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- added copper zone on F.Cu, net /Vcc
- added copper zone on B.Cu, net GND
Other:
- board outline added: 50.8 x 35.6 mm
- board text added: "2"
- board text added: "3"
- board text added: "4"
- board text added: "5"
- board text added: "6"
- board text added: "7"
- board text added: "8"
- board text added: "C2[22pF]"
- board text added: "C3"
- board text added: "C4[0.1uF]"
- board text added: "D1[LED]"
- board text added: "D2[LED]"
- board text added: "GND"
- board text added: "GPIO"
- board text added: "I2C"
- board text added: "ICSP"
- board text added: "MCU Data Logger For AtMega 328P - 2Mbit EEPROM - RTC - I2C, SPI, GPIOs"
- board text added: "MISO SCK RESET"
- board text added: "R3[4.7K]"
- board text added: "R4[4.7K]"
- board text added: "R5[330]"
- board text added: "R6[10K]"
- board text added: "R7[330]"
- board text added: "RX"
- board text added: "SCK"
- board text added: "SDA"
- board text added: "TX"
- board text added: "UART"
- board text added: "VCC"
- board text added: "VCC MOSI GND"
