File: Dattalogger_Board.kicad_pcb (KiCad board)
At the start: 2 copper layers, 50.8 x 35.6 mm, 30 parts, among them J1 Conn_01x04_Pin, J2 Conn_01x04_Pin, J3 Conn_02x03_Odd_Even, J4 Conn_01x09_Pin, U1 24LC1025, U2 DS1337S_, U3 24LC1025, U4 ATMega328P-AU, Y1 32.768 KHz, Y2 16 MHz

Commit message: Completed 3-layer pcb routing
Parts:
- moved Majed 1.80 mm to (161.9, 74.9)
- moved C3 0.16 mm to (152.4, 66.2)
Routing:
- net GND: track 184.6 -> 210.8 mm, vias 5 -> 14
- net /SCK: track 99.2 -> 124.4 mm, vias 3 -> 7
- net /Vcc: track 221.0 -> 242.3 mm, vias 7 -> 14
- net Net-(U4-AREF): track 21.1 -> 11.9 mm, vias 2 -> 0
- net /TX: track 29.0 -> 35.2 mm
- net /RX: track 27.1 -> 32.3 mm
- net Net-(U2-SQW/~INT): track 6.53 -> 11.4 mm
- net /MOSI: track 24.8 -> 29.2 mm, vias 0 -> 1
- net /D2: track 27.4 -> 30.3 mm, vias 1 -> 0
- net /D7: track 15.5 -> 12.8 mm, vias 1 -> 0
- net /D8: track 12.4 -> 13.8 mm, vias 1 -> 0
- net Net-(U4-PB7): track 31.5 -> 30.1 mm, vias 2 -> 3
- net Net-(U4-PB6): track 24.2 -> 23.0 mm, vias 0 -> 3
- net /D6: track 14.5 -> 13.5 mm, vias 1 -> 0
- net /D3: track 24.6 -> 25.5 mm
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- added copper zone on In1.Cu, net /Vcc
- removed copper zone on F.Cu, net /Vcc
Other:
- copper layers 2 -> 4

Commit message: Completed
Parts:
- moved Majed 1.42 mm to (161.3, 76.2)
Changed lines of the file:
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@@
       (drillshape 0)
       (scaleselection 1)
-      (outputdirectory "Datalogger_Gerbers/")
+      (outputdirectory "4_layer_MCU_Datalogger_Gerbers/")
     )
   )
@@
   )
   (footprint "Library2:MajedDev" (layer "B.Cu")
-    (at 161.925 74.93 180)
+    (at 161.29 76.2 180)
     (attr board_only exclude_from_pos_files exclude_from_bom)
     (fp_text reference "Majed" (at 0 0) (layer "B.SilkS") hide
