File: Dattalogger_Board.kicad_sch (KiCad schematic)
At the start: 25 parts, among them U1 24LC1025, U2 DS1337S_, U3 24LC1025, U4 ATMEGA328P-AU, Y1 32.768 KHz, Y2 16 MHz

Commit message: fixed bugs in schematic
Connections:
- net SCK: no longer R3.2, U1.6 (SCL), U2.6 (SCL), U3.6 (SCL), U4.28 (PC5)
- new net SCL: R3.2, U1.6 (SCL), U2.6 (SCL), U3.6 (SCL), U4.28 (PC5)
Other:
- sheet Connectors ports: added SCL; removed none
Changed lines of the file:
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@@
     (stroke (width 0) (type default))
   )
-  (wire (pts (xy 186.69 132.08) (xy 198.12 132.08))
+  (wire (pts (xy 187.96 147.32) (xy 198.12 147.32))
     (stroke (width 0) (type default))
   )
@@
   )
   (wire (pts (xy 185.42 43.18) (xy 193.04 43.18))
+    (stroke (width 0) (type default))
+  )
+  (wire (pts (xy 186.69 133.35) (xy 198.12 133.35))
     (stroke (width 0) (type default))
   )
@@
     (effects (font (size 1.27 1.27)) (justify left bottom))
   )
-  (label "SCK" (at 186.69 71.12 0) (fields_autoplaced)
+  (label "SCL" (at 186.69 71.12 0) (fields_autoplaced)
     (effects (font (size 1.27 1.27)) (justify left bottom))
   )
@@
     (effects (font (size 1.27 1.27)) (justify left bottom))
   )
-  (label "SCK" (at 38.1 44.45 0) (fields_autoplaced)
+  (label "SCL" (at 38.1 44.45 0) (fields_autoplaced)
     (effects (font (size 1.27 1.27)) (justify left bottom))
   )
@@
     (effects (font (size 1.27 1.27)) (justify left bottom))
   )
-  (label "SCK" (at 186.69 132.08 0) (fields_autoplaced)
+  (label "SCK" (at 187.96 147.32 0) (fields_autoplaced)
     (effects (font (size 1.27 1.27)) (justify left bottom))
   )
@@
     (effects (font (size 1.27 1.27)) (justify left bottom))
   )
+  (label "SCL" (at 186.69 133.35 0) (fields_autoplaced)
+    (effects (font (size 1.27 1.27)) (justify left bottom))
+  )
   (label "Vcc" (at 20.32 158.75 0) (fields_autoplaced)
     (effects (font (size 1.27 1.27)) (justify left bottom))
@@
     (effects (font (size 1.27 1.27)) (justify left bottom))
   )
-  (label "SCK" (at 50.8 156.21 0) (fields_autoplaced)
+  (label "SCL" (at 50.8 156.21 0) (fields_autoplaced)
     (effects (font (size 1.27 1.27)) (justify left bottom))
   )
@@
     (effects (font (size 1.27 1.27)) (justify left bottom))
   )
-  (label "SCK" (at 92.71 156.21 0) (fields_autoplaced)
+  (label "SCL" (at 92.71 156.21 0) (fields_autoplaced)
     (effects (font (size 1.27 1.27)) (justify left bottom))
   )
@@
     (effects (font (size 1.27 1.27)) (justify left bottom))
   )
-  (label "SCK" (at 106.68 168.91 0) (fields_autoplaced)
+  (label "SCL" (at 106.68 168.91 0) (fields_autoplaced)
     (effects (font (size 1.27 1.27)) (justify left bottom))
   )
@@
       (effects (font (size 1.27 1.27)) (justify left))
     )
-    (pin "SCK" passive (at 198.12 132.08 180)
+    (pin "SCK" passive (at 198.12 147.32 180)
       (effects (font (size 1.27 1.27)) (justify left))
     )
@@
       (effects (font (size 1.27 1.27)) (justify left))
     )
+    (pin "SCL" passive (at 198.12 133.35 180)
+      (effects (font (size 1.27 1.27)) (justify left))
+    )
